File: DigitalGuitarHub.kicad_sch (KiCad schematic)
At the start: 0 parts

Commit message: WIP
Parts:
- added C10, C11, C13, C16, C7, C8: 100nF, Capacitor_SMD:C_0402_1005Metric, symbol Device:C
- added C12, C2, C4, C9, C? (x2): 10uF, Capacitor_SMD:C_0805_2012Metric, symbol Device:C
- added C14: 1nF (NP0), symbol Device:C_Small
- added C15: 2.2nF (NP0), symbol Device:C_Small
- added C17: 10uF (Electrolyte), symbol Device:C_Polarized
- added C6: 100nF (NP0), symbol Device:C
- added D1: D_TVS, symbol Device:D_TVS
- added J1: USB_C_Receptacle, Connector_USB:USB_C_Receptacle_Molex_105450-0101, symbol Connector:USB_C_Receptacle
- added R1, R2: 27R, Resistor_SMD:R_0805_2012Metric, symbol Device:R
- added R10: 10k, symbol Device:R
- added R11, R8, R9: 4k7, symbol Device:R
- added R3, R4: 5k1 1%, Resistor_SMD:R_0603_1608Metric, symbol Device:R_Small
- added R5, R?: 1R, Resistor_SMD:R_0805_2012Metric, symbol Device:R
- added R6: 1k, Resistor_SMD:R_0603_1608Metric, symbol Device:R
- added R7: 1M, symbol Device:R
- added U1: AMS1117-3.3, Package_TO_SOT_SMD:SOT-223-3_TabPin2, symbol Regulator_Linear:AMS1117-3.3
- added U2, U4: OPA1671, Package_TO_SOT_SMD:SOT-353_SC-70-5, symbol DigitalGuiterHub_Lib:OPA1671
- added U3: PCM3060, Package_SO:TSSOP-28_4.4x9.7mm_P0.65mm, symbol Audio:PCM3060
- added U?: AMS1117-5.0, Package_TO_SOT_SMD:SOT-223-3_TabPin2, symbol Regulator_Linear:AMS1117-5.0
Connections:
- new net: C4.2, R5.1
- new net: C15.1, R8.2, R9.1
- new net: C14.1, R9.2, U4.3 (+)
- new net: C6.2, R6.2
- new net: C6.1, R7.2, U2.3 (+)
- new net: C15.2, C17.1, U4.1, U4.4 (-)
- new net: C17.2, R10.2
- new net: J1.A5 (CC1), R3.2
- new net: C?.2, R?.1
- new net: C8.1, U3.26 (V_{IN}R)
- new net: J1.A1 (GND), J1.A12 (GND), J1.B1 (GND), J1.B12 (GND), J1.S1 (SHIELD)
- new net: J1.A4 (VBUS), J1.A9 (VBUS), J1.B4 (VBUS), J1.B9 (VBUS)
- new net: J1.B5 (CC2), R4.2
- new net +2V5: C13.1, R7.1, U3.21 (V_{COM})
- new net +3V3: C10.1, C4.1, C9.1, C?.1, U1.2 (VO), U3.7 (V_{DD}), U?.2 (VO)
- new net +5V: C11.1, C12.1, C16.1, C7.1, U2.5 (V+), U3.24 (V_{CC}), U4.5 (V+)
- new net +VBUS: C2.1, C?.1, U1.3 (VI), U?.3 (VI)
- new net ADC_{DOUT}: U3.3 (DOUT)
- new net ADC_{IN}: U2.1, U2.4 (-), U3.25 (V_{IN}L)
- new net A_{IN}: D1.2 (A2), R6.1
- new net A_{OUT}: R10.1, R11.2
- new net CODEC_{~{RST}}: U3.15 (~{RST})
- new net DAC_{DIN}: U3.12 (DIN)
- new net DAC_{OUT}: R8.1, U3.20 (V_{OUT}L+)
- new net GND: C10.2, C11.2, C12.2, C13.2, C14.2, C16.2, C2.2, C7.2, C8.2, C9.2, C?.2, D1.1 (A1), R11.1, R3.1, R4.1, R5.2, R?.2, U1.1 (GND), U2.2 (V-), U3.16 (SGND), U3.22 (AGND2), U3.23 (AGND1), U3.8 (DGND), U4.2 (V-), U?.1 (GND)
- new net RP2350/USB_DN: R1.1
- new net RP2350/USB_DP: R2.1
- new net USB_DN: J1.A7 (D-), J1.B7 (D-), R1.2
- new net USB_DP: J1.A6 (D+), J1.B6 (D+), R2.2
- no-connect marks 0 -> 18
Other:
- added sheet LED ARRAY (Subsheets/LEDArray.kicad_sch)
- added sheet RP2350 (Subsheets/RP2350_minimal.kicad_sch)
- note added: "3V3 Digital power supply"
- note added: "5V Analog power supply"
- note added: "ADC & DAC"
- note added: "Input buffer"
- note added: "LED ARRAY"
- note added: "Output filter"
- note added: "RP2350A"
- note added: "USB-C"
- company: (none) -> by Daniel Siwiaszczyk
- title: (none) -> Digital Guitar Hub
